File: PCB/PCB.kicad_sch (KiCad schematic)
At the start: 0 parts

Commit message: its a gam console. idk thought it would be cool to make one
Parts:
- added BT1: Battery, symbol Device:Battery
- added D1: LED, symbol Device:LED
- added J1: Micro_SD_Card, symbol Connector:Micro_SD_Card
- added LS1: Speaker, symbol Device:Speaker
- added SW1, SW3, SW5, SW6, SW7, SW8: SW_Push, symbol Switch:SW_Push
- added SW2: SW_Slide_DPDT, symbol Switch:SW_Slide_DPDT
- added SW4: RotaryEncoder_Switch_MP, symbol Device:RotaryEncoder_Switch_MP
- added U1: Pico, RPi_Pico:RPi_Pico_SMD_TH, symbol Taranium-libs:Pico
- added U2: CR2013-MI2120, Display:CR2013-MI2120, symbol Driver_Display:CR2013-MI2120
- added U3: COM-09032, COM-09032:XDCR_COM-09032, symbol COM-09032:COM-09032
Connections:
- new net: SW1.1, SW6.1
- new net: SW1.2, SW3.2, SW5.2
- new net: SW6.2, SW7.2, SW8.2
- new net: SW5.1, SW8.1
- new net: SW3.1, SW7.1
- new net +3V3: U1.36 (3V3)
- new net GND: U1.38 (GND), U3.S1 (SHIELD), U3.S2 (SHIELD), U3.S3 (SHIELD), U3.S4 (SHIELD)
- new net VBUS: SW2.1 (A), U1.40 (VBUS)

Commit message: the firmware is scaring me. im gonna go back to drivng macropad
Parts:
- removed LS1: Speaker, symbol Device:Speaker
- removed SW4: RotaryEncoder_Switch_MP, symbol Device:RotaryEncoder_Switch_MP
- removed U3: COM-09032, COM-09032:XDCR_COM-09032, symbol COM-09032:COM-09032
- added J2: MAX98357A, symbol Connector:Conn_01x07_Pin
- added R1: R_Small, symbol Device:R_Small
- added SW10: RotaryEncoder_Switch_MP, symbol Device:RotaryEncoder_Switch_MP
- added SW4, SW9: SW_Push, symbol Switch:SW_Push
Connections:
- net +3V3: now also J1.4 (VDD), U2.1 (VCC), J2.7 (Pin_7)
- net GND: now also BT1.2 (-), D1.1 (K), J1.6 (VSS), J1.9 (SHIELD), SW1.2, SW3.2, SW5.2, SW6.2, SW7.2, SW8.2, U1.13 (GND), U1.18 (GND), U1.23 (GND), U1.28 (GND), U1.3 (GND), U1.33 (AGND), U1.8 (GND), U2.2 (GND), J2.6 (Pin_6), SW10.C, SW10.MP, SW10.S2, SW4.2, SW9.2
- net VBUS: now also R1.2; no longer SW2.1 (A)
- net +BATT: now reaches SW2.2 (B)
- net +BATT: now also BT1.1 (+)
- net CS: now reaches U2.3 (~{CS})
- net RESET: now reaches U2.4 (RESET)
- net DC: now reaches U2.5 (D/~{C})
- net MOSI: now reaches U2.6 (MOSI)
- net SCK: now reaches U2.7 (SCK)
- net LED: now reaches U2.8 (LED)
- net MISO: now reaches U2.9 (MISO)
- net VS: now reaches U1.39 (VSYS)
- net VS: now also SW2.1 (A)
- net START: now reaches SW6.1
- net START: no longer SW1.1
- net DAT2: now reaches J1.1 (DAT2)
- net DAT3: now reaches J1.2 (DAT3/CD)
- net CMD: now reaches J1.3 (CMD)
- net CLK: now reaches J1.5 (CLK)
- net DAT0: now reaches J1.7 (DAT0)
- net DAT1: now reaches J1.8 (DAT1)
- net at D1.2 (A): now also R1.1
- net A: now reaches SW8.1
- net A: no longer SW5.1
- net DOWN: now reaches SW3.1
- net DOWN: no longer SW7.1
- new net B: SW9.1
- new net BCLK: J2.2 (Pin_2)
- new net DIN: J2.3 (Pin_3)
- new net ENC_A: SW10.A
- new net ENC_B: SW10.B
- new net GAIN: J2.4 (Pin_4)
- new net LEFT: SW4.1
- new net LRC: J2.1 (Pin_1)
- new net MENU: SW7.1
- new net MUTE: SW10.S1
- new net RIGHT: SW5.1
- new net SD: J2.5 (Pin_5)
- new net UP: SW1.1
Other:
- moved on the sheet: BT1, D1, SW1, SW2

Commit message: ingore
Parts:
- added RV1: R_Potentiometer_MountingPin, Package_SO:TSSOP-20_4.4x6.5mm_P0.65mm, symbol Device:R_Potentiometer_MountingPin
Changed lines of the file:
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@@
+	)
+	(symbol
+		(lib_id "Device:R_Potentiometer_MountingPin")
+		(at 73.66 78.74 0)
+		(unit 1)
+		(exclude_from_sim no)
+		(in_bom yes)
+		(on_board yes)
+		(dnp no)
+		(fields_autoplaced yes)
+		(property "Reference" "RV1"
+			(at 91.44 72.3198 0)
+			(effects
+				(font
+					(size 1.27 1.27)
+				)
+			)
+		)
+		(property "Value" "R_Potentiometer_MountingPin"
+			(at 91.44 74.8598 0)
+			(effects
+				(font
+					(size 1.27 1.27)
+				)
+			)
+		)
+		(property "Footprint" "Package_SO:TSSOP-20_4.4x6.5mm_P0.65mm"
+			(at 73.66 78.74 0)
+			(effects
+				(font
+					(size 1.27 1.27)
+				)
+				(hide yes)
+			)
+		)
+		(property "Datasheet" "~"
+			(at 73.66 78.74 0)
+			(effects
+				(font
+					(size 1.27 1.27)
+				)
+				(hide yes)
+			)
+		)
+		(property "Description" "Potentiometer with a mounting pin"
+			(at 73.66 78.74 0)
+			(effects
+				(font
+					(size 1.27 1.27)
+				)
+				(hide yes)
+			)
+		)
+		(pin "1"
+		)
+		(pin "3"
+		)
+		(pin "2"
+		)
+		(pin "MP"
+		)
+		(instances
+			(project ""
+				(path "/3f06ce5a-2ea1-4d36-9589-43839d98e41e"
+					(reference "RV1")
+					(unit 1)
+				)
+			)
+		)
 	)
 	(symbol

Commit message: commit
Parts:
- removed SW10: RotaryEncoder_Switch_MP, symbol Device:RotaryEncoder_Switch_MP
- added J3: AMP Output, symbol Connector:Conn_01x02_Pin
- BT1, SW2: footprint (none) -> Connector_PinHeader_2.54mm:PinHeader_1x02_P2.54mm_Vertical
- D1: footprint (none) -> LED_THT:LED_D3.0mm
- J1: footprint (none) -> Connector_Card:microSD_HC_Hirose_DM3AT-SF-PEJM5
- J2: footprint (none) -> Connector_PinHeader_2.54mm:PinHeader_1x06_P2.54mm_Vertical
- R1: footprint (none) -> Resistor_THT:R_Axial_DIN0204_L3.6mm_D1.6mm_P5.08mm_Horizontal
- RV1: footprint Package_SO:TSSOP-20_4.4x6.5mm_P0.65mm -> (none)
- SW1, SW3, SW4, SW5, SW6, SW7, SW8, SW9: footprint (none) -> Taranium-libs:Button-6mm-2pin-tht
- U1: footprint RPi_Pico:RPi_Pico_SMD_TH -> Module:RaspberryPi_Pico_Common_SMD
- U2: footprint Display:CR2013-MI2120 -> Connector_PinHeader_2.54mm:PinHeader_1x09_P2.54mm_Vertical
Connections:
- net GND: now also RV1.1, RV1.MP (MountPin)
- net AMP+: now reaches RV1.2
- net at RV1.3: now also J3.1 (Pin_1)
- new net AMP-: J3.2 (Pin_2)
Other:
- moved on the sheet: J2, RV1, U2
